Commit message: control

File: franka_description/robots/common/franka_arm.gazebo.xacro (robot description, xacro)
@@ -117,4 +117,10 @@
       <child link="${arm_id}_link8"/>
     </joint>
+    <link name="${arm_id}_ee"/>
+    <joint name="${arm_id}_ee" type="fixed">
+      <origin rpy="0 0 ${-pi/4}" xyz="0 0 0.2104"/>
+      <parent link="${arm_id}_link7"/>
+      <child link="${arm_id}_ee"/>
+    </joint>
     <!-- Collision sensors on all links. This is not present on the real robot, it is used only in simulation to detect collisions. -->
     <gazebo reference="${arm_id}_link1">
@@ -209,30 +215,4 @@
       </sensor>
     </gazebo>
-    <gazebo reference="${arm_id}_leftfinger">
-      <sensor name='${arm_id}_leftfinger_contact' type='contact'>
-        <update_rate> 50 </update_rate>
-        <always_on>true</always_on>
-          <contact>
-              <collision>${arm_id}_leftfinger_collision</collision>
-          </contact>
-          <plugin name="leftfinger_bumper" filename="libgazebo_ros_bumper.so">
-            <bumperTopicName>${arm_id}_leftfinger_collision</bumperTopicName>
-            <frameName>${arm_id}_leftfinger</frameName>
-          </plugin>
-      </sensor>
-    </gazebo>
-    <gazebo reference="${arm_id}_rightfinger">
-        <sensor name='${arm_id}_rightfinger_contact' type='contact'>
-          <update_rate> 50 </update_rate>
-          <always_on>true</always_on>
-            <contact>
-                <collision>${arm_id}_rightfinger_collision</collision>
-            </contact>
-            <plugin name="rightfinger_bumper" filename="libgazebo_ros_bumper.so">
-              <bumperTopicName>${arm_id}_rightfinger_collision</bumperTopicName>
-              <frameName>${arm_id}_rightfinger</frameName>
-            </plugin>
-        </sensor>
-      </gazebo>
   </xacro:macro>
 </robot>

File: franka_description/robots/common/franka_robot.gazebo.xacro (robot description, xacro)
@@ -6,5 +6,5 @@
     <xacro:franka_arm arm_id="${arm_id}" safety_distance="0.03" gazebo="${gazebo}" joint_limits="${joint_limits}"/>
     <xacro:if value="${hand}">
-      <xacro:include filename="$(find franka_description)/robots/common/franka_hand.xacro"/>
+      <xacro:include filename="$(find franka_description)/robots/common/franka_hand.gazebo.xacro"/>
       <xacro:franka_hand
           arm_id="${arm_id}"

Commit message: fix collision box

File: franka_description/robots/common/franka_arm.gazebo.xacro (robot description, xacro)
@@ -123,96 +123,96 @@
       <child link="${arm_id}_ee"/>
     </joint>
-    <!-- Collision sensors on all links. This is not present on the real robot, it is used only in simulation to detect collisions. -->
     <gazebo reference="${arm_id}_link1">
-      <sensor name='${arm_id}_link1_contact' type='contact'>
-        <update_rate> 50 </update_rate>
-        <always_on>true</always_on>
-          <contact>
+        <sensor name='${arm_id}_link1_contact' type='contact'>
+          <update_rate> 50 </update_rate>
+          <always_on>true</always_on>
+            <contact>
               <collision>${arm_id}_link1_collision</collision>
-          </contact>
-          <plugin name="link1_bumper" filename="libgazebo_ros_bumper.so">
-            <bumperTopicName>${arm_id}_link1_collision</bumperTopicName>
-            <frameName>${arm_id}_link1</frameName>
-          </plugin>
-      </sensor>
-    </gazebo>
-    <gazebo reference="${arm_id}_link2">
-      <sensor name='${arm_id}_link2_contact' type='contact'>
-        <update_rate> 50 </update_rate>
-        <always_on>true</always_on>
-          <contact>
+            </contact>
+            <plugin name="link1_bumper" filename="libgazebo_ros_bumper.so">
+              <bumperTopicName>${arm_id}_link1_collision</bumperTopicName>
+              <frameName>${arm_id}_link1</frameName>
+            </plugin>
+        </sensor>
+      </gazebo>
+      <gazebo reference="${arm_id}_link2">
+        <sensor name='${arm_id}_link2_contact' type='contact'>
+          <update_rate> 50 </update_rate>
+          <always_on>true</always_on>
+            <contact>
               <collision>${arm_id}_link2_collision</collision>
-          </contact>
-          <plugin name="link2_bumper" filename="libgazebo_ros_bumper.so">
-            <bumperTopicName>${arm_id}_link2_collision</bumperTopicName>
-            <frameName>${arm_id}_link2</frameName>
-          </plugin>
-      </sensor>
-    </gazebo>
-    <gazebo reference="${arm_id}_link3">
-      <sensor name='${arm_id}_link3_contact' type='contact'>
-        <update_rate> 50 </update_rate>
-        <always_on>true</always_on>
-          <contact>
+            </contact>
+            <plugin name="link2_bumper" filename="libgazebo_ros_bumper.so">
+              <bumperTopicName>${arm_id}_link2_collision</bumperTopicName>
+              <frameName>${arm_id}_link2</frameName>
+            </plugin>
+        </sensor>
+      </gazebo>
+      <gazebo reference="${arm_id}_link3">
+        <sensor name='${arm_id}_link3_contact' type='contact'>
+          <update_rate> 50 </update_rate>
+          <always_on>true</always_on>
+            <contact>
               <collision>${arm_id}_link3_collision</collision>
-          </contact>
-          <plugin name="link3_bumper" filename="libgazebo_ros_bumper.so">
-            <bumperTopicName>${arm_id}_link3_collision</bumperTopicName>
-            <frameName>${arm_id}_link3</frameName>
-          </plugin>
-      </sensor>
-    </gazebo>
-    <gazebo reference="${arm_id}_link4">
-      <sensor name='${arm_id}_link4_contact' type='contact'>
-        <update_rate> 50 </update_rate>
-        <always_on>true</always_on>
-          <contact>
+            </contact>
+            <plugin name="link3_bumper" filename="libgazebo_ros_bumper.so">
+              <bumperTopicName>${arm_id}_link3_collision</bumperTopicName>
+              <frameName>${arm_id}_link3</frameName>
+            </plugin>
+        </sensor>
+      </gazebo>
+      <gazebo reference="${arm_id}_link4">
+        <sensor name='${arm_id}_link4_contact' type='contact'>
+          <update_rate> 50 </update_rate>
+          <always_on>true</always_on>
+            <contact>
               <collision>${arm_id}_link4_collision</collision>
-          </contact>
-          <plugin name="link4_bumper" filename="libgazebo_ros_bumper.so">
-            <bumperTopicName>${arm_id}_link4_collision</bumperTopicName>
-            <frameName>${arm_id}_link4</frameName>
-          </plugin>
-      </sensor>
-    </gazebo>
-    <gazebo reference="${arm_id}_link5">
-      <sensor name='${arm_id}_link5_contact' type='contact'>
-        <update_rate> 50 </update_rate>
-        <always_on>true</always_on>
-          <contact>
+            </contact>
+            <plugin name="link4_bumper" filename="libgazebo_ros_bumper.so">
+              <bumperTopicName>${arm_id}_link4_collision</bumperTopicName>
+              <frameName>${arm_id}_link4</frameName>
+            </plugin>
+        </sensor>
+      </gazebo>
+      <gazebo reference="${arm_id}_link5">
+        <sensor name='${arm_id}_link5_contact' type='contact'>
+          <update_rate> 50 </update_rate>
+          <always_on>true</always_on>
+            <contact>
               <collision>${arm_id}_link5_collision</collision>
-          </contact>
-          <plugin name="link5_bumper" filename="libgazebo_ros_bumper.so">
-            <bumperTopicName>${arm_id}_link5_collision</bumperTopicName>
-            <frameName>${arm_id}_link5</frameName>
-          </plugin>
-      </sensor>
-    </gazebo>
-    <gazebo reference="${arm_id}_link6">
-      <sensor name='${arm_id}_link6_contact' type='contact'>
-        <update_rate> 50 </update_rate>
-        <always_on>true</always_on>
-          <contact>
+            </contact>
+            <plugin name="link5_bumper" filename="libgazebo_ros_bumper.so">
+              <bumperTopicName>${arm_id}_link5_collision</bumperTopicName>
+              <frameName>${arm_id}_link5</frameName>
+            </plugin>
+        </sensor>
+      </gazebo>
+      <gazebo reference="${arm_id}_link6">
+        <sensor name='${arm_id}_link6_contact' type='contact'>
+          <update_rate> 50 </update_rate>
+          <always_on>true</always_on>
+            <contact>
               <collision>${arm_id}_link6_collision</collision>
-          </contact>
-          <plugin name="link6_bumper" filename="libgazebo_ros_bumper.so">
-            <bumperTopicName>${arm_id}_link6_collision</bumperTopicName>
-            <frameName>${arm_id}_link6</frameName>
-          </plugin>
-      </sensor>
-    </gazebo>
-    <gazebo reference="${arm_id}_link7">
-      <sensor name='${arm_id}_link7_contact' type='contact'>
-        <update_rate> 50 </update_rate>
-        <always_on>true</always_on>
-          <contact>
+            </contact>
+            <plugin name="link6_bumper" filename="libgazebo_ros_bumper.so">
+              <bumperTopicName>${arm_id}_link6_collision</bumperTopicName>
+              <frameName>${arm_id}_link6</frameName>
+            </plugin>
+        </sensor>
+      </gazebo>
+      <gazebo reference="${arm_id}_link7">
+        <sensor name='${arm_id}_link7_contact' type='contact'>
+          <update_rate> 50 </update_rate>
+          <always_on>true</always_on>
+            <contact>
               <collision>${arm_id}_link7_collision</collision>
-          </contact>
-          <plugin name="link7_bumper" filename="libgazebo_ros_bumper.so">
-            <bumperTopicName>${arm_id}_link7_collision</bumperTopicName>
-            <frameName>${arm_id}_link7</frameName>
-          </plugin>
-      </sensor>
-    </gazebo>
+              <collision>${arm_id}_link7_fixed_joint_lump__panda_hand_collision_1</collision>
+            </contact>
+            <plugin name="link7_bumper" filename="libgazebo_ros_bumper.so">
+              <bumperTopicName>${arm_id}_link7_collision</bumperTopicName>
+              <frameName>${arm_id}_link7</frameName>
+            </plugin>
+        </sensor>
+      </gazebo>
   </xacro:macro>
 </robot>

File: franka_description/robots/common/franka_hand.gazebo.xacro (robot description, xacro)
@@ -117,23 +117,42 @@
       <dynamics damping="0.3" />
     </joint>
-    <gazebo reference="${arm_id}_leftfinger">
+    <!-- <gazebo reference="${arm_id}_hand">
       <sensor name='${arm_id}_leftfinger_contact' type='contact'>
         <update_rate> 50 </update_rate>
         <always_on>true</always_on>
           <contact>
-              <collision>${arm_id}_leftfinger_collision</collision>
+              <collision>${arm_id}_hand_collision</collision>
           </contact>
-          <plugin name="leftfinger_bumper" filename="libgazebo_ros_bumper.so">
-            <bumperTopicName>${arm_id}_leftfinger_collision</bumperTopicName>
-            <frameName>${arm_id}_leftfinger</frameName>
+          <plugin name="hand_bumper" filename="libgazebo_ros_bumper.so">
+            <bumperTopicName>${arm_id}_hand_collision</bumperTopicName>
+            <frameName>${arm_id}_hand</frameName>
           </plugin>
       </sensor>
-    </gazebo>
-    <gazebo reference="${arm_id}_rightfinger">
+    </gazebo> -->
+    <gazebo reference="${arm_id}_leftfinger">
+        <sensor name='${arm_id}_leftfinger_contact' type='contact'>
+          <update_rate> 50 </update_rate>
+          <always_on>true</always_on>
+            <contact>
+              <collision>${arm_id}_leftfinger_collision</collision>
+              <collision>${arm_id}_leftfinger_collision_1</collision>
+              <collision>${arm_id}_leftfinger_collision_2</collision>
+              <collision>${arm_id}_leftfinger_collision_3</collision>
+            </contact>
+            <plugin name="leftfinger_bumper" filename="libgazebo_ros_bumper.so">
+              <bumperTopicName>${arm_id}_leftfinger_collision</bumperTopicName>
+              <frameName>${arm_id}_leftfinger</frameName>
+            </plugin>
+        </sensor>
+      </gazebo>
+      <gazebo reference="${arm_id}_rightfinger">
         <sensor name='${arm_id}_rightfinger_contact' type='contact'>
           <update_rate> 50 </update_rate>
           <always_on>true</always_on>
             <contact>
-                <collision>${arm_id}_rightfinger_collision</collision>
+              <collision>${arm_id}_rightfinger_collision</collision>
+              <collision>${arm_id}_rightfinger_collision_1</collision>
+              <collision>${arm_id}_rightfinger_collision_2</collision>
+              <collision>${arm_id}_rightfinger_collision_3</collision>
             </contact>
             <plugin name="rightfinger_bumper" filename="libgazebo_ros_bumper.so">
@@ -142,5 +161,5 @@
             </plugin>
         </sensor>
-    </gazebo>
+      </gazebo>
   </xacro:macro>
 </robot>

File: franka_description/robots/common/franka_robot.gazebo.xacro (robot description, xacro)
@@ -70,4 +70,19 @@
         <self_collide>true</self_collide>
       </gazebo>
+      <!-- Collision sensors on all links. This is not present on the real robot, it is used only in simulation to detect collisions. -->
+      <!--  -->
+      <!-- <gazebo reference="${arm_id}_link8">
+        <sensor name='${arm_id}_link8_contact' type='contact'>
+          <update_rate> 50 </update_rate>
+          <always_on>true</always_on>
+            <contact>
+              <collision>${arm_id}_link8_collision</collision>
+            </contact>
+            <plugin name="link8_bumper" filename="libgazebo_ros_bumper.so">
+              <bumperTopicName>${arm_id}_link8_collision</bumperTopicName>
+              <frameName>${arm_id}_link8</frameName>
+            </plugin>
+        </sensor>
+      </gazebo> -->
     </xacro:if>
   </xacro:macro>
